File: altimeter.sch (EAGLE design)
At the start: 22 parts, among them U1 DPS310, U2 WT51822-S4ATMODULE, U3 MMA8452Q, U4 MIC5205-3.3YM5-TR

Commit message: Silkscreen cleanup before gerber export.
Parts:
- renumbered X1 to USB
Changed lines of the file:
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@@
 <part name="+3V10" library="supply1" library_urn="urn:adsk.eagle:library:371" deviceset="+3V3" device=""/>
 <part name="GND11" library="supply1" library_urn="urn:adsk.eagle:library:371" deviceset="GND" device=""/>
-<part name="X1" library="Testing" deviceset="USB-AB" device="IN&amp;OUT"/>
+<part name="USB" library="Testing" deviceset="USB-AB" device="IN&amp;OUT"/>
 <part name="GND3" library="SparkFun" deviceset="GND" device=""/>
 <part name="GND12" library="SparkFun" deviceset="GND" device=""/>
@@
 <instance part="+3V10" gate="G$1" x="111.76" y="142.24"/>
 <instance part="GND11" gate="1" x="109.22" y="111.76"/>
-<instance part="X1" gate="G$1" x="175.26" y="160.02" rot="R180"/>
+<instance part="USB" gate="G$1" x="175.26" y="160.02" rot="R180"/>
 <instance part="GND3" gate="1" x="185.42" y="147.32"/>
 <instance part="GND12" gate="1" x="228.6" y="137.16"/>
@@
 </segment>
 <segment>
-<pinref part="X1" gate="G$1" pin="GND"/>
+<pinref part="USB" gate="G$1" pin="GND"/>
 <pinref part="GND3" gate="1" pin="GND"/>
 <wire x1="180.34" y1="154.94" x2="185.42" y2="154.94" width="0.1524" layer="91"/>
@@
 <segment>
 <pinref part="R1" gate="G$1" pin="1"/>
-<pinref part="X1" gate="G$1" pin="VBUS"/>
+<pinref part="USB" gate="G$1" pin="VBUS"/>
 <wire x1="187.96" y1="165.1" x2="180.34" y2="165.1" width="0.1524" layer="91"/>
 </segment>
@@
 <net name="DP" class="0">
 <segment>
-<pinref part="X1" gate="G$1" pin="D+"/>
+<pinref part="USB" gate="G$1" pin="D+"/>
 <wire x1="180.34" y1="160.02" x2="193.04" y2="160.02" width="0.1524" layer="91"/>
 <label x="213.36" y="160.02" size="1.27" layer="95" font="vector" xref="yes"/>
@@
 <net name="DM" class="0">
 <segment>
-<pinref part="X1" gate="G$1" pin="D-"/>
+<pinref part="USB" gate="G$1" pin="D-"/>
 <wire x1="180.34" y1="162.56" x2="200.66" y2="162.56" width="0.1524" layer="91"/>
 <label x="213.36" y="162.56" size="1.27" layer="95" font="vector" xref="yes"/>
